Commit message: added gps

File: urdf/robot.urdf.xacro (robot description, xacro)
@@ -17,3 +17,4 @@
     <!-- <xacro:include filename="depth_camera.xacro"/> -->
     <xacro:include filename="imu.xacro"/>
+    <xacro:include filename="gps.xacro"/>
 </robot>

File: urdf/sensors/imu.xacro (robot description, xacro)
@@ -40,4 +40,5 @@
         <pose>0 0 0 0 0 0</pose>
       </sensor>
+      <material>Gazebo/Orange</material>
     </gazebo>
 </robot>

Commit message: UWB plugin working

File: urdf/robot.urdf.xacro (robot description, xacro)
@@ -17,4 +17,5 @@
     <!-- <xacro:include filename="depth_camera.xacro"/> -->
     <xacro:include filename="imu.xacro"/>
-    <xacro:include filename="gps.xacro"/>
+    <!-- <xacro:include filename="gps.xacro"/> -->
+    <xacro:include filename="uwb.xacro"/>
 </robot>

File: urdf/sensors/depth_camera.xacro (robot description, xacro)
@@ -11,5 +11,5 @@
                 <box size="0.010 0.03 0.03"/>
             </geometry>
-            <material name="red"/>
+            <material name="orange"/>
         </visual>
     </link>
@@ -21,5 +21,5 @@
     <link name="camera_link_optical"></link>
     <gazebo reference="camera_link">
-        <material>Gazebo/Red</material>
+        <material>Gazebo/Orange</material>
         <sensor name="camera" type="depth">
             <pose> 0 0 0 0 0 0 </pose>
